File: colibri_hw/esp_core.kicad_sch (KiCad schematic)
At the start: 10 parts

Commit message: [v1.0.1]: Fix UART communication issues due to R5 value
Parts:
- C2: value (none) -> 100n; footprint (none) -> Capacitor_SMD:C_1206_3216Metric
- R3, R4, R6, R8: value (none) -> 10k; footprint (none) -> Resistor_SMD:R_0805_2012Metric
- R5: value (none) -> R*; footprint (none) -> Resistor_SMD:R_0805_2012Metric
- R7: value (none) -> 4.7k; footprint (none) -> Resistor_SMD:R_0805_2012Metric
- R9: value (none) -> 1k; footprint (none) -> Resistor_SMD:R_0805_2012Metric
- U1: value (none) -> ESP-12E; footprint (none) -> ESP8266:ESP-12E_SMD
- U2: value (none) -> DS18B20; footprint (none) -> Package_TO_SOT_THT:TO-92
Other:
- note added: "*Optional do not mount"
Changed lines of the file:
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@@
     (stroke (width 0) (type default) (color 0 0 0 0))
   )
+  (text "*Optional\ndo not mount" (at 180.34 73.66 0)
+    (effects (font (size 1.27 1.27)) (justify left bottom))
+  )
   (global_label "gpio2" (shape input) (at 171.45 92.71 0) (fields_autoplaced)
     (effects (font (size 1.27 1.27)) (justify left))
@@
       (effects (font (size 1.27 1.27)) (justify left))
     )
-    (property "Value" "" (id 1) (at 128.651 104.013 0)
-      (effects (font (size 1.27 1.27)) (justify left))
-    )
-    (property "Footprint" "" (id 2) (at 126.6952 106.68 0)
+    (property "Value" "100n" (id 1) (at 128.651 104.013 0)
+      (effects (font (size 1.27 1.27)) (justify left))
+    )
+    (property "Footprint" "Capacitor_SMD:C_1206_3216Metric" (id 2) (at 126.6952 106.68 0)
       (effects (font (size 1.27 1.27)) hide)
     )
@@
       (effects (font (size 1.27 1.27)) hide)
     )
-    (property "Value" "" (id 1) (at 125.857 111.0742 0))
+    (property "Value" "GND" (id 1) (at 125.857 111.0742 0))
     (property "Footprint" "" (id 2) (at 125.73 106.68 0)
       (effects (font (size 1.27 1.27)) hide)
@@
       (effects (font (size 1.27 1.27)) (justify left))
     )
-    (property "Value" "" (id 1) (at 109.728 70.993 0)
-      (effects (font (size 1.27 1.27)) (justify left))
-    )
-    (property "Footprint" "" (id 2) (at 106.172 69.85 90)
+    (property "Value" "10k" (id 1) (at 109.728 70.993 0)
+      (effects (font (size 1.27 1.27)) (justify left))
+    )
+    (property "Footprint" "Resistor_SMD:R_0805_2012Metric" (id 2) (at 106.172 69.85 90)
       (effects (font (size 1.27 1.27)) hide)
     )
@@
     (in_bom yes) (on_board yes)
     (property "Reference" "U1" (id 0) (at 148.59 68.199 0))
-    (property "Value" "" (id 1) (at 148.59 70.5104 0))
-    (property "Footprint" "" (id 2) (at 148.59 87.63 0)
+    (property "Value" "ESP-12E" (id 1) (at 148.59 70.5104 0))
+    (property "Footprint" "ESP8266:ESP-12E_SMD" (id 2) (at 148.59 87.63 0)
       (effects (font (size 1.27 1.27)) hide)
     )
@@
       (effects (font (size 1.27 1.27)) hide)
     )
-    (property "Value" "" (id 1) (at 171.577 102.1842 0))
+    (property "Value" "GND" (id 1) (at 171.577 102.1842 0))
     (property "Footprint" "" (id 2) (at 171.45 97.79 0)
       (effects (font (size 1.27 1.27)) hide)
@@
       (effects (font (size 1.27 1.27)) (justify right))
     )
-    (property "Value" "" (id 1) (at 243.332 88.773 0)
+    (property "Value" "DS18B20" (id 1) (at 243.332 88.773 0)
       (effects (font (size 1.27 1.27)) (justify right))
     )
-    (property "Footprint" "" (id 2) (at 262.89 93.98 0)
+    (property "Footprint" "Package_TO_SOT_THT:TO-92" (id 2) (at 262.89 93.98 0)
       (effects (font (size 1.27 1.27)) hide)
     )
@@
       (effects (font (size 1.27 1.27)) (justify left))
     )
-    (property "Value" "" (id 1) (at 127.508 70.993 0)
-      (effects (font (size 1.27 1.27)) (justify left))
-    )
-    (property "Footprint" "" (id 2) (at 123.952 69.85 90)
+    (property "Value" "10k" (id 1) (at 127.508 70.993 0)
+      (effects (font (size 1.27 1.27)) (justify left))
+    )
+    (property "Footprint" "Resistor_SMD:R_0805_2012Metric" (id 2) (at 123.952 69.85 90)
       (effects (font (size 1.27 1.27)) hide)
     )
@@
       (effects (font (size 1.27 1.27)) (justify left))
     )
-    (property "Value" "" (id 1) (at 177.038 107.823 0)
-      (effects (font (size 1.27 1.27)) (justify left))
-    )
-    (property "Footprint" "" (id 2) (at 173.482 106.68 90)
+    (property "Value" "10k" (id 1) (at 177.038 107.823 0)
+      (effects (font (size 1.27 1.27)) (justify left))
+    )
+    (property "Footprint" "Resistor_SMD:R_0805_2012Metric" (id 2) (at 173.482 106.68 90)
       (effects (font (size 1.27 1.27)) hide)
     )
@@
       (effects (font (size 1.27 1.27)) (justify right))
     )
-    (property "Value" "" (id 1) (at 225.552 82.423 0)
+    (property "Value" "4.7k" (id 1) (at 225.552 82.423 0)
       (effects (font (size 1.27 1.27)) (justify right))
     )
-    (property "Footprint" "" (id 2) (at 225.552 81.28 90)
+    (property "Footprint" "Resistor_SMD:R_0805_2012Metric" (id 2) (at 225.552 81.28 90)
       (effects (font (size 1.27 1.27)) hide)
     )
@@
       (effects (font (size 1.27 1.27)) hide)
     )
-    (property "Value" "" (id 1) (at 175.387 114.8842 0))
+    (property "Value" "GND" (id 1) (at 175.387 114.8842 0))
     (property "Footprint" "" (id 2) (at 175.26 110.49 0)
       (effects (font (size 1.27 1.27)) hide)
@@
       (effects (font (size 1.27 1.27)) hide)
     )
-    (property "Value" "" (id 1) (at 237.617 99.6442 0))
+    (property "Value" "GND" (id 1) (at 237.617 99.6442 0))
     (property "Footprint" "" (id 2) (at 237.49 95.25 0)
       (effects (font (size 1.27 1.27)) hide)
@@
     (in_bom yes) (on_board yes)
     (property "Reference" "R5" (id 0) (at 175.26 65.8622 90))
-    (property "Value" "" (id 1) (at 175.26 68.1736 90))
-    (property "Footprint" "" (id 2) (at 175.26 72.898 90)
+    (property "Value" "R*" (id 1) (at 175.26 68.1736 90))
+    (property "Footprint" "Resistor_SMD:R_0805_2012Metric" (id 2) (at 175.26 72.898 90)
       (effects (font (size 1.27 1.27)) hide)
     )
@@
       (effects (font (size 1.27 1.27)) (justify left))
     )
-    (property "Value" "" (id 1) (at 237.998 35.433 0)
-      (effects (font (size 1.27 1.27)) (justify left))
-    )
-    (property "Footprint" "" (id 2) (at 234.442 34.29 90)
+    (property "Value" "10k" (id 1) (at 237.998 35.433 0)
+      (effects (font (size 1.27 1.27)) (justify left))
+    )
+    (property "Footprint" "Resistor_SMD:R_0805_2012Metric" (id 2) (at 234.442 34.29 90)
       (effects (font (size 1.27 1.27)) hide)
     )
@@
       (effects (font (size 1.27 1.27)) (justify left))
     )
-    (property "Value" "" (id 1) (at 237.998 48.133 0)
-      (effects (font (size 1.27 1.27)) (justify left))
-    )
-    (property "Footprint" "" (id 2) (at 234.442 46.99 90)
+    (property "Value" "1k" (id 1) (at 237.998 48.133 0)
+      (effects (font (size 1.27 1.27)) (justify left))
+    )
+    (property "Footprint" "Resistor_SMD:R_0805_2012Metric" (id 2) (at 234.442 46.99 90)
       (effects (font (size 1.27 1.27)) hide)
     )
@@
       (effects (font (size 1.27 1.27)) hide)
     )
-    (property "Value" "" (id 1) (at 236.347 55.1942 0))
+    (property "Value" "GND" (id 1) (at 236.347 55.1942 0))
     (property "Footprint" "" (id 2) (at 236.22 50.8 0)
       (effects (font (size 1.27 1.27)) hide)
